Commit message: <second_commit>

File: robot/robot_description/urdf/robot_description.urdf (robot description, URDF)
Before this commit: robot robot_description, 8 links, 7 joints
Links:
- removed link lidar_link
- added link base_scan, mass 0.073085; collision mesh filename=package://robot_description/meshes/lidar_link.STL; visual mesh filename=package://robot_description/meshes/lidar_link.STL
Joints:
- joint base_joint: origin xyz=0 0 0.010 rpy=0 0 0 -> xyz=0 0 0.0005 rpy=0 0 0
- joint lidar_joint: child lidar_link -> base_scan
